File: KiCad/TRax-Controller/TRax-Controller.sch (KiCad schematic (older format))
At the start: 37 parts, among them J1 Inputs, J2 BldgPwr, J3 Outputs, J5 Grove LCD, J6 Raspberry Pi Header, U1 4N25, U2 4N25, U3 4N25, U4 4N25, U5 4N25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

Commit message: bumped schematic version, cleaned up
Parts:
- J6: symbol TRax-RaspberryPi-rescue:Raspberry_Pi_TRax-myLib -> TRax-Controller-rescue:Raspberry_Pi_TRax-myLib-TRax-RaspberryPi-rescue
Changed lines of the file:
@@
 $EndComp
 $Comp
-L TRax-RaspberryPi-rescue:Raspberry_Pi_TRax-myLib J6
+L TRax-Controller-rescue:Raspberry_Pi_TRax-myLib-TRax-RaspberryPi-rescue J6
 U 1 1 6089B0A9
 P 8500 3500
@@
 	8500 2000 8500 2100
 Connection ~ 8500 2100
-Entry Wire Line
-	1600 0    1700 100
 $EndSCHEMATC
