File: KiCad/TRax-Relays/TRax-Relays.sch (KiCad schematic (older format))
At the start: 14 parts, among them J1 WX, J10 Relays, J2 RoofPower, J3 MountPower, J4 Open/Close, J5 Parked, J6 Fob, J7 Inputs, J8 Relays, J9 Conn_01x08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

Commit message: switch to 6P6C connectors; misc cleanup
Parts:
- J1, J2, J3, J4, J5, J6: symbol Connector:6P4C -> Connector:6P6C
Connections:
- net at J1.2: no longer J7.1 (Pin_1)
- net at J1.4: now also J2.4, J3.4, J4.2, J4.4, J5.4, J7.8 (Pin_8)
- net at J3.2: now also J2.2, J6.3, J8.1 (Pin_1); no longer J7.3 (Pin_3)
- net at J8.3 (Pin_3): now also J3.5; no longer J3.4
- net at J7.2 (Pin_2): now also J2.3; no longer J2.2
- net at J8.2 (Pin_2): now also J2.5; no longer J2.4
- net at J7.4 (Pin_4): now also J4.3; no longer J4.2
- net at J7.5 (Pin_5): now also J4.5; no longer J4.4
- net at J5.2: now also J6.2, J8.7 (Pin_7); no longer J7.6 (Pin_6)
- net at J8.5 (Pin_5): now also J5.5; no longer J5.4
- net at J8.4 (Pin_4): now also J6.4; no longer J6.3
- net at J8.6 (Pin_6): now also J6.5; no longer J6.4
- net at K1.~ (VCC): now also J10.2 (Pin_2)
- net at K2.~ (VCC): now also J10.3 (Pin_3)
- net at K3.~ (VCC): now also J10.4 (Pin_4)
- new net: J1.3, J7.1 (Pin_1)
- new net: J3.3, J7.3 (Pin_3)
- new net: J5.3, J7.6 (Pin_6)
- new net: K1.~ (VCC), K2.~ (VCC), K3.~ (VCC), K4.~ (VCC) (x2)
- new net: J10.1 (Pin_1), K1.~ (VCC), K2.~ (VCC), K3.~ (VCC)
- now unconnected: J2.1, J3.1, J4.1, J5.1, J6.1
- no-connect marks 7 -> 19
Other:
- note added: "RJ Color Code: Telco (Cat5)\n5. Yellow (Orange/White)\n4. Green (White/Blue)\n3. Red (Blue/White)\n2. Black (White/Orange"
- note added: "black"
- note added: "blue"
- note added: "green"
- note added: "orange"
- note added: "red"
- note added: "violet"
- note added: "white"
- note added: "yellow"
- note removed: "RJ Color Code: Telco (Cat5)\n4. Yellow (Orange/White)\n3. Green (White/Blue)\n2. Red (Blue/White)\n1. Black (White/Orange"
Changed lines of the file:
@@
 encoding utf-8
 Sheet 1 1
-Title "Relays & Connector wiring"
-Date "2021-05-09"
-Rev "v1.2"
+Title "T-Rax Relays & Connector wiring"
+Date "2021-05-22"
+Rev "v1.2b"
 Comp "Robert Ferguson Observatory"
 Comment1 "David Kensiski"
@@
 Green
 $Comp
-L Connector:6P4C J1
+L Connector:6P6C J1
 U 1 1 609A144B
 P 1600 1600
@@
 $EndComp
 $Comp
-L Connector:6P4C J3
+L Connector:6P6C J3
 U 1 1 609A2420
 P 1600 3600
@@
 $EndComp
 $Comp
-L Connector:6P4C J2
+L Connector:6P6C J2
 U 1 1 609A2BC1
 P 1600 2600
@@
 $EndComp
 $Comp
-L Connector:6P4C J4
+L Connector:6P6C J4
 U 1 1 609A37E0
 P 1600 4600
@@
 $EndComp
 $Comp
-L Connector:6P4C J5
+L Connector:6P6C J5
 U 1 1 609A462B
 P 1600 5600
@@
 $EndComp
 Text Notes 1050 7550 0    50   ~ 0
-RJ Color Code: Telco (Cat5)\n4. Yellow (Orange/White)\n3. Green  (White/Blue)\n2. Red    (Blue/White)\n1. Black  (White/Orange
+RJ Color Code: Telco (Cat5)\n5. Yellow (Orange/White)\n4. Green  (White/Blue)\n3. Red    (Blue/White)\n2. Black  (White/Orange
 Wire Wire Line
 	2000 1600 3150 1600
@@
 	5950 4700 5600 4700
 $Comp
-L Connector:6P4C J6
+L Connector:6P6C J6
 U 1 1 609A546C
 P 1600 6600
@@
 	1    0    0    -1
 $EndComp
-Text Notes 2650 5400 2    50   ~ 0
+Text Notes 3400 5400 2    50   ~ 0
 12V switched
 Wire Wire Line
@@
 	5100 3400 5500 3400
 Wire Wire Line
-	5500 3400 5500 5400
-Wire Wire Line
 	4150 3400 4150 5400
 Wire Wire Line
 	2000 6700 4350 6700
-Wire Wire Line
-	5400 7100 5400 5500
-Wire Wire Line
-	5400 5500 5950 5500
-Wire Wire Line
-	5400 5500 5400 3500
-Connection ~ 5400 5500
 Wire Wire Line
 	5100 3500 5400 3500
@@
 Wire Wire Line
 	4250 3500 4250 6400
-Text Notes 2250 6400 2    50   ~ 0
+Text Notes 3050 6400 2    50   ~ 0
 12V\n
 Wire Wire Line
@@
 Wire Wire Line
 	5100 3000 5850 3000
-Wire Wire Line
-	5500 5400 5950 5400
 Wire Notes Line
 	8850 2350 8850 5750
@@
 Wire Bus Line
 	5350 1950 10100 1950
+NoConn ~ 2000 6300
+NoConn ~ 2000 6800
+NoConn ~ 2000 5800
+NoConn ~ 2000 5300
+NoConn ~ 2000 4800
+NoConn ~ 2000 4300
+NoConn ~ 2000 3800
+NoConn ~ 2000 3300
+NoConn ~ 2000 2800
+NoConn ~ 2000 2300
+NoConn ~ 2000 1800
+NoConn ~ 2000 1300
+Text Notes 2200 6700 0    50   ~ 0
+black
+Text Notes 2200 6600 0    50   ~ 0
+blue
+Text Notes 2200 6500 0    50   ~ 0
+yellow
+Text Notes 2200 6400 0    50   ~ 0
+red
+Text Notes 2200 5700 0    50   ~ 0
+black
+Text Notes 2200 4700 0    50   ~ 0
+black
+Text Notes 2200 3500 0    50   ~ 0
+black
+Text Notes 2200 2700 0    50   ~ 0
+blue
+Text Notes 2200 1600 0    50   ~ 0
+violet
+Text Notes 2200 5600 0    50   ~ 0
+white
+Text Notes 2200 5500 0    50   ~ 0
+black
+Text Notes 2200 5400 0    50   ~ 0
+white
+Text Notes 2200 4600 0    50   ~ 0
+orange
+Text Notes 2200 4500 0    50   ~ 0
+black
+Text Notes 2200 4400 0    50   ~ 0
+yellow
+Text Notes 2200 3600 0    50   ~ 0
+green
+Text Notes 2200 3700 0    50   ~ 0
+blue
+Text Notes 2200 3400 0    50   ~ 0
+orange
+Text Notes 2200 2600 0    50   ~ 0
+blue
+Text Notes 2200 2500 0    50   ~ 0
+black
+Text Notes 2200 2400 0    50   ~ 0
+green
+Text Notes 2200 1500 0    50   ~ 0
+black
+Wire Wire Line
+	5400 3500 5400 5400
+Wire Wire Line
+	5500 5500 5950 5500
+Wire Wire Line
+	5500 3400 5500 5500
+Wire Wire Line
+	5950 5400 5400 5400
+Wire Bus Line
+	7950 2450 10100 2450
 Wire Bus Line
 	5250 1150 5250 1850
-Wire Bus Line
-	7950 2450 10100 2450
+Connection ~ 5400 5400
+Wire Wire Line
+	5400 5400 5400 7100
 $EndSCHEMATC

Commit message: pulled custom relay symbol into library
Parts:
- K1, K2, K3, K4: symbol myLib:Relay_Module -> TRax-Relays-rescue:Relay_Module-myLib
Connections:
- net at K1.~ (VCC): now also J10.2 (Pin_2)
- net at K2.~ (VCC): now also J10.3 (Pin_3)
- net at K3.~ (VCC): now also J10.4 (Pin_4)
- new net: K1.~ (VCC), K2.~ (VCC), K3.~ (VCC), K4.~ (VCC) (x2)
- new net: J10.1 (Pin_1), K1.~ (VCC), K2.~ (VCC), K3.~ (VCC)
Changed lines of the file:
@@
 $EndComp
 $Comp
-L myLib:Relay_Module K1
+L TRax-Relays-rescue:Relay_Module-myLib K1
 U 1 1 609A763A
 P 6400 2950
@@
 $EndComp
 $Comp
-L myLib:Relay_Module K2
+L TRax-Relays-rescue:Relay_Module-myLib K2
 U 1 1 609A9B89
 P 6400 3750
@@
 $EndComp
 $Comp
-L myLib:Relay_Module K3
+L TRax-Relays-rescue:Relay_Module-myLib K3
 U 1 1 609AA6A6
 P 6400 4550
@@
 $EndComp
 $Comp
-L myLib:Relay_Module K4
+L TRax-Relays-rescue:Relay_Module-myLib K4
 U 1 1 609AAFF2
 P 6400 5350
@@
 Wire Wire Line
 	5950 5400 5400 5400
+Connection ~ 5400 5400
+Wire Wire Line
+	5400 5400 5400 7100
 Wire Bus Line
 	7950 2450 10100 2450
 Wire Bus Line
 	5250 1150 5250 1850
-Connection ~ 5400 5400
-Wire Wire Line
-	5400 5400 5400 7100
 $EndSCHEMATC

Commit message: fix red/black wiring on input RJ11s
Connections:
- net at J1.4, J2.4, J3.4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: now also J7.7 (Pin_7); no longer J7.8 (Pin_8)
- net at K1.~ (VCC): now also J10.2 (Pin_2)
- net at K2.~ (VCC): now also J10.3 (Pin_3)
- net at K3.~ (VCC): now also J10.4 (Pin_4)
- new net: K1.~ (VCC), K2.~ (VCC), K3.~ (VCC), K4.~ (VCC) (x2)
- new net: J10.1 (Pin_1), K1.~ (VCC), K2.~ (VCC), K3.~ (VCC)
- no-connect marks 19 -> 18
Other:
- note added: "* The red leads (+3.3v) on these jacks are wired to “black” pins.\n I had wired them with black (ground) initially but that turned out to\n be in error and it was easier to just change the color than rewire\n the whole thing."
- note added: "red*"
Changed lines of the file:
@@
 Sheet 1 1
 Title "T-Rax Relays & Connector wiring"
-Date "2021-05-22"
-Rev "v1.2b"
+Date "2021-07-14"
+Rev "v1.3"
 Comp "Robert Ferguson Observatory"
 Comment1 "David Kensiski"
 Comment2 ""
 Comment3 ""
-Comment4 ""
+Comment4 "v1.3 fixes black/red wiring on input RJ11s"
 $EndDescr
 Text Notes 4500 1050 2    50   ~ 0
@@
 Wire Wire Line
 	3650 1550 4550 1550
-NoConn ~ 4550 1650
 Wire Wire Line
 	3650 1550 3650 5600
@@
 	3150 1050 4550 1050
 Wire Wire Line
-	3050 1500 3050 1750
-Wire Wire Line
 	2000 5500 3050 5500
 Wire Wire Line
 	2000 1500 3050 1500
-Wire Wire Line
-	4550 1750 3050 1750
-Connection ~ 3050 1750
-Wire Wire Line
-	3050 1750 3050 2500
 Wire Wire Line
 	2000 2500 3050 2500
@@
 Text Notes 2200 6400 0    50   ~ 0
 red
-Text Notes 2200 5700 0    50   ~ 0
-black
 Text Notes 2200 4700 0    50   ~ 0
-black
+red*
 Text Notes 2200 3500 0    50   ~ 0
-black
+red*
 Text Notes 2200 2700 0    50   ~ 0
 blue
@@
 white
 Text Notes 2200 5500 0    50   ~ 0
-black
+red*
 Text Notes 2200 5400 0    50   ~ 0
 white
@@
 orange
 Text Notes 2200 4500 0    50   ~ 0
-black
+red*
 Text Notes 2200 4400 0    50   ~ 0
 yellow
@@
 blue
 Text Notes 2200 2500 0    50   ~ 0
-black
+red*
 Text Notes 2200 2400 0    50   ~ 0
 green
 Text Notes 2200 1500 0    50   ~ 0
-black
+red*
 Wire Wire Line
 	5400 3500 5400 5400
@@
 Wire Wire Line
 	5400 5400 5400 7100
+Wire Wire Line
+	4550 1650 3750 1650
+Wire Wire Line
+	3750 1750 3050 1750
+Connection ~ 3050 1750
+Wire Wire Line
+	3050 1750 3050 2500
+Wire Wire Line
+	3750 1650 3750 1750
+Wire Wire Line
+	3050 1500 3050 1750
 Wire Bus Line
 	7950 2450 10100 2450
 Wire Bus Line
 	5250 1150 5250 1850
+Text Notes 2200 5700 0    50   ~ 0
+black
+Text Notes 1050 7950 0    50   ~ 0
+* The red leads (+3.3v) on these jacks are wired to “black” pins.\n   I had wired them with black (ground) initially but that turned out to\n   be in error and it was easier to just change the color than rewire\n   the whole thing.
 $EndSCHEMATC
