File: KiCad/TRax-Schematic/TRax-Controller.sch (KiCad schematic (older format))
At the start: 37 parts, among them J1 Inputs, J2 BldgPwr, J3 Outputs, J5 Grove LCD, J6 Raspberry Pi Header, U1 4N25, U2 4N25, U3 4N25, U4 4N25, U5 4N25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

Commit message: merged all there schematics into one
Parts:
- J6: symbol TRax-Controller-rescue:Raspberry_Pi_TRax-myLib-TRax-RaspberryPi-rescue -> TRax-Controller-rescue:Raspberry_Pi_TRax-myLib-TRax-RaspberryPi-rescue-TRax-Controller-rescue
Changed lines of the file:
@@
 $Descr A 11000 8500
 encoding utf-8
-Sheet 1 1
+Sheet 1 3
 Title "T-Rax Control Board"
 Date "2021-05-06"
@@
 $EndComp
 $Comp
-L TRax-Controller-rescue:Raspberry_Pi_TRax-myLib-TRax-RaspberryPi-rescue J6
+L TRax-Controller-rescue:Raspberry_Pi_TRax-myLib-TRax-RaspberryPi-rescue-TRax-Controller-rescue J6
 U 1 1 6089B0A9
 P 8500 3500
@@
 L power:PWR_FLAG #FLG0101
 U 1 1 608D0375
-P 5350 7300
-F 0 "#FLG0101" H 5350 7375 50  0001 C CNN
-F 1 "PWR_FLAG" H 5350 7473 50  0000 C CNN
-F 2 "" H 5350 7300 50  0001 C CNN
-F 3 "~" H 5350 7300 50  0001 C CNN
-	1    5350 7300
+P 11550 7800
+F 0 "#FLG0101" H 11550 7875 50  0001 C CNN
+F 1 "PWR_FLAG" H 11550 7973 50  0000 C CNN
+F 2 "" H 11550 7800 50  0001 C CNN
+F 3 "~" H 11550 7800 50  0001 C CNN
+	1    11550 7800
 	1    0    0    -1
 $EndComp
@@
 L power:PWR_FLAG #FLG0102
 U 1 1 608D1C6B
-P 5650 7300
-F 0 "#FLG0102" H 5650 7375 50  0001 C CNN
-F 1 "PWR_FLAG" H 5650 7473 50  0000 C CNN
-F 2 "" H 5650 7300 50  0001 C CNN
-F 3 "~" H 5650 7300 50  0001 C CNN
-	1    5650 7300
+P 11850 7800
+F 0 "#FLG0102" H 11850 7875 50  0001 C CNN
+F 1 "PWR_FLAG" H 11850 7973 50  0000 C CNN
+F 2 "" H 11850 7800 50  0001 C CNN
+F 3 "~" H 11850 7800 50  0001 C CNN
+	1    11850 7800
 	-1   0    0    1
 $EndComp
@@
 L power:+3.3V #PWR0131
 U 1 1 608D2B2B
-P 5650 7300
-F 0 "#PWR0131" H 5650 7150 50  0001 C CNN
-F 1 "+3.3V" H 5665 7473 50  0000 C CNN
-F 2 "" H 5650 7300 50  0001 C CNN
-F 3 "" H 5650 7300 50  0001 C CNN
-	1    5650 7300
+P 11850 7800
+F 0 "#PWR0131" H 11850 7650 50  0001 C CNN
+F 1 "+3.3V" H 11865 7973 50  0000 C CNN
+F 2 "" H 11850 7800 50  0001 C CNN
+F 3 "" H 11850 7800 50  0001 C CNN
+	1    11850 7800
 	1    0    0    -1
 $EndComp
@@
 L power:GND #PWR0132
 U 1 1 608D3AD7
-P 5350 7300
-F 0 "#PWR0132" H 5350 7050 50  0001 C CNN
-F 1 "GND" H 5355 7127 50  0000 C CNN
-F 2 "" H 5350 7300 50  0001 C CNN
-F 3 "" H 5350 7300 50  0001 C CNN
-	1    5350 7300
+P 11550 7800
+F 0 "#PWR0132" H 11550 7550 50  0001 C CNN
+F 1 "GND" H 11555 7627 50  0000 C CNN
+F 2 "" H 11550 7800 50  0001 C CNN
+F 3 "" H 11550 7800 50  0001 C CNN
+	1    11550 7800
 	1    0    0    -1
 $EndComp
@@
 L power:PWR_FLAG #FLG0103
 U 1 1 60A1CC87
-P 5950 7300
-F 0 "#FLG0103" H 5950 7375 50  0001 C CNN
-F 1 "PWR_FLAG" H 5950 7473 50  0000 C CNN
-F 2 "" H 5950 7300 50  0001 C CNN
-F 3 "~" H 5950 7300 50  0001 C CNN
-	1    5950 7300
+P 12150 7800
+F 0 "#FLG0103" H 12150 7875 50  0001 C CNN
+F 1 "PWR_FLAG" H 12150 7973 50  0000 C CNN
+F 2 "" H 12150 7800 50  0001 C CNN
+F 3 "~" H 12150 7800 50  0001 C CNN
+	1    12150 7800
 	1    0    0    1
 $EndComp
@@
 L power:+5V #PWR0130
 U 1 1 60A2A59E
-P 5950 7300
-F 0 "#PWR0130" H 5950 7150 50  0001 C CNN
-F 1 "+5V" H 5965 7473 50  0000 C CNN
-F 2 "" H 5950 7300 50  0001 C CNN
-F 3 "" H 5950 7300 50  0001 C CNN
-	1    5950 7300
+P 12150 7800
+F 0 "#PWR0130" H 12150 7650 50  0001 C CNN
+F 1 "+5V" H 12165 7973 50  0000 C CNN
+F 2 "" H 12150 7800 50  0001 C CNN
+F 3 "" H 12150 7800 50  0001 C CNN
+	1    12150 7800
 	1    0    0    -1
 $EndComp
@@
 	8500 2000 8500 2100
 Connection ~ 8500 2100
+$Sheet
+S 11700 700  1150 400
+U 6146FF07
+F0 "TRax Relays" 50
+F1 "TRax-Relays.sch" 50
+$EndSheet
+$Sheet
+S 11700 2250 1150 350
+U 61524F60
+F0 "TRax Laser Park Detector" 50
+F1 "TRax-LaserParkDetector.sch" 50
+$EndSheet
 $EndSCHEMATC
